File: keypie/keypie.kicad_pcb (KiCad board)
At the start: 2 copper layers, 16 x 45 mm, 36 parts, among them J1 USB_C_Receptacle_USB2.0_14P, J2 USB_C_Receptacle_USB2.0_14P, SW1 SW_Push, U1 SPX3819M5-L-3-3, U2 W25Q64JVXGIQ, U3 W25Q64JVXGIQ, U4 ABM8-272-T3_C20625731, U5 RP2040

Commit message: better work or else
Parts:
- R5, R6: value 5.1k -> 56k
- moved R6 1.34 mm to (110.2, 135.9)
- moved R5 1.08 mm to (105.1, 136.1)
Connections:
- R5 pad 2: GND -> VCC
- R6 pad 1: GND -> VCC
Routing:
- net VCC: track 61.2 -> 65.4 mm
- net Net-(J2-CC1): track 3.47 -> 2.40 mm
Changed lines of the file:
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@@
 			)
 		)
-		(property "Datasheet" "~"
+		(property "Datasheet" ""
 			(at 0 0 45)
 			(layer "F.Fab")
@@
 			)
 		)
-		(property "Datasheet" "~"
+		(property "Datasheet" ""
 			(at 0 0 45)
 			(layer "F.Fab")
@@
 			)
 		)
-		(property "Datasheet" "~"
+		(property "Datasheet" ""
 			(at 0 0 45)
 			(layer "F.Fab")
@@
 			)
 		)
-		(property "Datasheet" "~"
+		(property "Datasheet" ""
 			(at 0 0 0)
 			(layer "F.Fab")
@@
 			)
 		)
-		(property "Datasheet" "~"
+		(property "Datasheet" ""
 			(at 0 0 135)
 			(layer "F.Fab")
@@
 			)
 		)
-		(property "Datasheet" "~"
+		(property "Datasheet" ""
 			(at 0 0 45)
 			(layer "F.Fab")
@@
 			)
 		)
-		(property "Datasheet" "~"
+		(property "Datasheet" ""
 			(at 0 0 90)
 			(layer "F.Fab")
@@
 			)
 		)
-		(property "Datasheet" "~"
+		(property "Datasheet" ""
 			(at 0 0 0)
 			(layer "F.Fab")
@@
 			)
 		)
-		(property "Datasheet" "~"
+		(property "Datasheet" ""
 			(at 0 0 45)
 			(layer "F.Fab")
@@
 			)
 		)
-		(property "Datasheet" "~"
+		(property "Datasheet" ""
 			(at 0 0 45)
 			(layer "F.Fab")
@@
 			)
 		)
-		(property "Datasheet" "~"
+		(property "Datasheet" ""
 			(at 0 0 45)
 			(layer "F.Fab")
@@
 			)
 		)
-		(property "Datasheet" "~"
+		(property "Datasheet" ""
 			(at 0 0 45)
 			(layer "F.Fab")
@@
 			)
 		)
-		(property "Datasheet" "~"
+		(property "Datasheet" ""
 			(at 0 0 0)
 			(layer "F.Fab")
@@
 			)
 		)
-		(property "Datasheet" "~"
+		(property "Datasheet" ""
 			(at 0 0 0)
 			(layer "F.Fab")
@@
 			)
 		)
-		(property "Datasheet" "~"
+		(property "Datasheet" ""
 			(at 0 0 135)
 			(layer "F.Fab")
@@
 			)
 		)
-		(property "Datasheet" "~"
+		(property "Datasheet" ""
 			(at 0 0 45)
 			(layer "F.Fab")
@@
 			)
 		)
-		(property "Datasheet" "~"
+		(property "Datasheet" ""
 			(at 0 0 45)
 			(layer "F.Fab")
@@
 			)
 		)
-		(property "Datasheet" "~"
+		(property "Datasheet" ""
 			(at 0 0 90)
 			(layer "F.Fab")
@@
 			)
 		)
-		(property "JLC_3DModel_Q" "370c585f985f42a3bbd3c7d32eb22fcc"
-			(at 0 0 0)
-			(layer "Cmts.User")
-			(hide yes)
-			(effects
-				(font
-					(size 1.27 1.27)
-					(thickness 0.15)
-				)
-			)
-		)
-		(property "JLC_3D_Size" "4.02 4"
-			(at 0 0 0)
-			(layer "Cmts.User")
-			(hide yes)
-			(effects
-				(font
-					(size 1.27 1.27)
-					(thickness 0.15)
-				)
-			)
-		)
 		(property ki_fp_filters "WSON*1EP*8x6mm*P1.27mm*")
 		(sheetname "/")
@@
 			)
 		)
-		(property "Datasheet" "~"
+		(property "Datasheet" ""
 			(at 0 0 0)
 			(layer "F.Fab")
@@
 			)
 		)
-		(property "JLC_3DModel_Q" "370c585f985f42a3bbd3c7d32eb22fcc"
-			(at 0 0 90)
-			(layer "Cmts.User")
-			(hide yes)
-			(effects
-				(font
-					(size 1.27 1.27)
-					(thickness 0.15)
-				)
-			)
-		)
-		(property "JLC_3D_Size" "4.02 4"
-			(at 0 0 90)
-			(layer "Cmts.User")
-			(hide yes)
-			(effects
-				(font
-					(size 1.27 1.27)
-					(thickness 0.15)
-				)
-			)
-		)
 		(property ki_fp_filters "WSON*1EP*8x6mm*P1.27mm*")
 		(sheetname "/")
@@
 			)
 		)
-		(property "Datasheet" "~"
+		(property "Datasheet" ""
 			(at 0 0 0)
 			(layer "F.Fab")
@@
 			)
 		)
-		(property "Datasheet" "~"
+		(property "Datasheet" ""
 			(at 0 0 45)
 			(layer "F.Fab")
@@
 			)
 		)
-		(property "Datasheet" "~"
+		(property "Datasheet" ""
 			(at 0 0 0)
 			(layer "F.Fab")
@@
 	(footprint "Capacitor_SMD:C_0402_1005Metric"
 		(layer "F.Cu")
-		(at 111.52 136.1 180)
+		(at 110.2 135.89 180)
 		(descr "Capacitor SMD 0402 (1005 Metric), square (rectangular) end terminal, IPC-7351 nominal, (Body size source: IPC-SM-782 page 76, https://www.pcb-3d.com/wordpress/wp-content/uploads/ipc-sm-782a_amendment_1_and_2.pdf), generated with kicad-footprint-generator")
 		(tags "capacitor")
 		(property "Reference" "R6"
-			(at -1.98 0.2 180)
+			(at -1.98 0.2 0)
 			(layer "F.SilkS")
 			(effects
@@
 			)
 		)
-		(property "Value" "5.1k"
+		(property "Value" "56k"
 			(at 0 1.16 0)
 			(layer "F.Fab")
@@
 			)
 		)
-		(property "Datasheet" "~"
+		(property "Datasheet" ""
 			(at 0 0 0)
 			(layer "F.Fab")
@@
 			(layers "F.Cu" "F.Mask" "F.Paste")
 			(roundrect_rratio 0.25)
-			(net 2 "GND")
+			(net 19 "VCC")
 			(pintype "passive")
 		)
@@
 			)
 		)
-		(property "Datasheet" "~"
+		(property "Datasheet" ""
 			(at 0 0 90)
 			(layer "F.Fab")
@@
 			)
 		)
-		(property "Datasheet" "~"
+		(property "Datasheet" ""
 			(at 0 0 0)
 			(layer "F.Fab")
@@
 			)
 		)
-		(property "Datasheet" "~"
+		(property "Datasheet" ""
 			(at 0 0 135)
 			(layer "F.Fab")
@@
 			)
 		)
-		(property "Datasheet" "~"
+		(property "Datasheet" ""
 			(at 0 0 0)
 			(layer "F.Fab")
@@
 			)
 		)
-		(property "Datasheet" "~"
+		(property "Datasheet" ""
 			(at 0 0 45)
 			(layer "F.Fab")
@@
 			(net 59 "unconnected-(U5-GPIO18-Pad29)")
 			(pinfunction "GPIO18")
-			(pintype "bidirectional")
+			(pintype "bidirectional+no_connect")
 		)
 		(pad "30" smd roundrect
@@
 			(net 60 "unconnected-(U5-GPIO19-Pad30)")
 			(pinfunction "GPIO19")
-			(pintype "bidirectional")
+			(pintype "bidirectional+no_connect")
 		)
 		(pad "31" smd roundrect
@@
 	(footprint "Capacitor_SMD:C_0402_1005Metric"
 		(layer "F.Cu")
-		(at 104.02 136 180)
+		(at 105.1 136.1 180)
 		(descr "Capacitor SMD 0402 (1005 Metric), square (rectangular) end terminal, IPC-7351 nominal, (Body size source: IPC-SM-782 page 76, https://www.pcb-3d.com/wordpress/wp-content/uploads/ipc-sm-782a_amendment_1_and_2.pdf), generated with kicad-footprint-generator")
 		(tags "capacitor")
@@
 			)
 		)
-		(property "Value" "5.1k"
+		(property "Value" "56k"
 			(at 0 1.16 0)
 			(layer "F.Fab")
@@
 			)
 		)
-		(property "Datasheet" "~"
+		(property "Datasheet" ""
 			(at 0 0 0)
 			(layer "F.Fab")
@@
 			(layers "F.Cu" "F.Mask" "F.Paste")
 			(roundrect_rratio 0.25)
-			(net 2 "GND")
+			(net 19 "VCC")
 			(pintype "passive")
 		)
@@
 	)
 	(segment
+		(start 110.45 137.855)
+		(end 110.45 136.12)
+		(width 0.4)
+		(layer "F.Cu")
+		(net 19)
+	)
+	(segment
 		(start 105.55 137.855)
 		(end 105.55 138.55)
@@
 	)
 	(segment
+		(start 105.55 137.855)
+		(end 105.55 137.03)
+		(width 0.4)
+		(layer "F.Cu")
+		(net 19)
+	)
+	(segment
+		(start 105.55 137.03)
+		(end 104.62 136.1)
+		(width 0.4)
+		(layer "F.Cu")
+		(net 19)
+	)
+	(segment
 		(start 114.702 132.35)
 		(end 113.45 132.35)
@@
 	)
 	(segment
+		(start 110.45 136.12)
+		(end 110.68 135.89)
+		(width 0.4)
+		(layer "F.Cu")
+		(net 19)
+	)
+	(segment
 		(start 113.1 132.7)
 		(end 113.1 133.4)
@@
 	)
 	(segment
-		(start 106.272 136.6)
-		(end 106.75 137.078)
-		(width 0.2)
-		(layer "F.Cu")
-		(net 25)
-	)
-	(segment
-		(start 105.1 136.6)
-		(end 106.272 136.6)
+		(start 106.75 136.990001)
+		(end 106.75 137.855)
 		(width 0.2)
 		(layer "F.Cu")
@@
 	)
 	(segment
-		(start 104.5 136)
-		(end 105.1 136.6)
+		(start 105.58 136.1)
+		(end 105.859999 136.1)
 		(width 0.2)
 		(layer "F.Cu")
@@
 	)
 	(segment
-		(start 106.75 137.078)
-		(end 106.75 137.855)
+		(start 105.859999 136.1)
+		(end 106.75 136.990001)
 		(width 0.2)
 		(layer "F.Cu")
@@
 	)
 	(segment
-		(start 109.75 137.128)
-		(end 109.75 137.855)
-		(width 0.2)
-		(layer "F.Cu")
-		(net 26)
-	)
-	(segment
-		(start 110.778 136.1)
-		(end 109.75 137.128)
+		(start 109.75 135.92)
+		(end 109.72 135.89)
 		(width 0.2)
 		(layer "F.Cu")
@@
 	)
 	(segment
-		(start 111.02 136.1)
-		(end 110.778 136.1)
+		(start 109.75 137.855)
+		(end 109.75 135.92)
 		(width 0.2)
 		(layer "F.Cu")
