File: keypie/keypie.kicad_sch (KiCad schematic)
At the start: 36 parts, among them J1 USB_C_Receptacle_USB2.0_14P, J2 USB_C_Receptacle_USB2.0_14P, SW1 SW_Push, U1 SPX3819M5-L-3-3, U2 W25Q64JVXGIQ, U3 W25Q64JVXGIQ, U4 ABM8-272-T3_C20625731, U5 RP2040

Commit message: better work or else
Parts:
- R5, R6: value 5.1k -> 56k
Connections:
- net GND: no longer R5.2, R6.1
- net VCC: now also R5.2, R6.1
- no-connect marks 25 -> 27
Other:
- note added: "Change to pull ups!!"
Changed lines of the file:
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@@
 		)
 	)
+	(text "Change to pull ups!!"
+		(exclude_from_sim no)
+		(at 131.826 73.152 0)
+		(effects
+			(font
+				(size 1.27 1.27)
+			)
+		)
+	)
 	(junction
 		(at 180.34 21.59)
@@
 	)
 	(junction
-		(at 113.03 74.93)
-		(diameter 0)
-		(color 0 0 0 0)
-	)
-	(junction
 		(at 223.52 27.94)
 		(diameter 0)
@@
 	)
 	(junction
+		(at 113.03 74.93)
+		(diameter 0)
+		(color 0 0 0 0)
+	)
+	(junction
 		(at 52.07 186.69)
 		(diameter 0)
@@
 	)
 	(no_connect
+		(at 217.17 99.06)
+	)
+	(no_connect
 		(at 41.91 30.48)
 	)
 	(no_connect
+		(at 217.17 101.6)
+	)
+	(no_connect
 		(at 91.44 176.53)
 	)
@@
 	(wire
 		(pts
-			(xy 113.03 73.66) (xy 113.03 74.93)
-		)
-		(stroke
-			(width 0)
-			(type default)
-		)
-	)
-	(wire
-		(pts
 			(xy 189.23 43.18) (xy 189.23 45.72)
 		)
@@
 	(wire
 		(pts
-			(xy 113.03 74.93) (xy 115.57 74.93)
-		)
-		(stroke
-			(width 0)
-			(type default)
-		)
-	)
-	(wire
-		(pts
 			(xy 232.41 27.94) (xy 232.41 29.21)
 		)
@@
 	(wire
 		(pts
-			(xy 113.03 74.93) (xy 113.03 76.2)
+			(xy 113.03 73.66) (xy 113.03 74.93)
 		)
 		(stroke
@@
 	(wire
 		(pts
+			(xy 113.03 74.93) (xy 113.03 76.2)
+		)
+		(stroke
+			(width 0)
+			(type default)
+		)
+	)
+	(wire
+		(pts
 			(xy 142.24 186.69) (xy 152.4 186.69)
 		)
@@
 	(wire
 		(pts
+			(xy 119.38 74.93) (xy 119.38 73.66)
+		)
+		(stroke
+			(width 0)
+			(type default)
+		)
+	)
+	(wire
+		(pts
 			(xy 201.93 43.18) (xy 199.39 43.18)
 		)
@@
 		)
 	)
+	(wire
+		(pts
+			(xy 113.03 74.93) (xy 119.38 74.93)
+		)
+		(stroke
+			(width 0)
+			(type default)
+		)
+	)
 	(polyline
 		(pts
@@
 	)
 	(symbol
+		(lib_id "power:VCC")
+		(at 119.38 73.66 0)
+		(unit 1)
+		(exclude_from_sim no)
+		(in_bom yes)
+		(on_board yes)
+		(dnp no)
+		(property "Reference" "#PWR017"
+			(at 119.38 77.47 0)
+			(effects
+				(font
+					(size 1.27 1.27)
+				)
+				(hide yes)
+			)
+		)
+		(property "Value" "VCC"
+			(at 119.38 70.358 0)
+			(effects
+				(font
+					(size 1.27 1.27)
+				)
+			)
+		)
+		(property "Footprint" ""
+			(at 119.38 73.66 0)
+			(effects
+				(font
+					(size 1.27 1.27)
+				)
+				(hide yes)
+			)
+		)
+		(property "Datasheet" ""
+			(at 119.38 73.66 0)
+			(effects
+				(font
+					(size 1.27 1.27)
+				)
+				(hide yes)
+			)
+		)
+		(property "Description" "Power symbol creates a global label with name \"VCC\""
+			(at 119.38 73.66 0)
+			(effects
+				(font
+					(size 1.27 1.27)
+				)
+				(hide yes)
+			)
+		)
+		(pin "1"
+		)
+		(instances
+			(project "keypie"
+				(path "/abc4a181-bf3c-43d0-89e8-0b6073fb1e2a"
+					(reference "#PWR017")
+					(unit 1)
+				)
+			)
+		)
+	)
+	(symbol
 		(lib_id "Device:R_Small")
 		(at 53.34 78.74 270)
@@
 	)
 	(symbol
-		(lib_id "power:GND")
-		(at 115.57 74.93 0)
-		(unit 1)
-		(exclude_from_sim no)
-		(in_bom yes)
-		(on_board yes)
-		(dnp no)
-		(fields_autoplaced yes)
-		(property "Reference" "#PWR017"
-			(at 115.57 81.28 0)
-			(effects
-				(font
-					(size 1.27 1.27)
-				)
-				(hide yes)
-			)
-		)
-		(property "Value" "GND"
-			(at 115.57 80.01 0)
-			(effects
-				(font
-					(size 1.27 1.27)
-				)
-			)
-		)
-		(property "Footprint" ""
-			(at 115.57 74.93 0)
-			(effects
-				(font
-					(size 1.27 1.27)
-				)
-				(hide yes)
-			)
-		)
-		(property "Datasheet" ""
-			(at 115.57 74.93 0)
-			(effects
-				(font
-					(size 1.27 1.27)
-				)
-				(hide yes)
-			)
-		)
-		(property "Description" "Power symbol creates a global label with name \"GND\" , ground"
-			(at 115.57 74.93 0)
-			(effects
-				(font
-					(size 1.27 1.27)
-				)
-				(hide yes)
-			)
-		)
-		(pin "1"
-		)
-		(instances
-			(project "keypie"
-				(path "/abc4a181-bf3c-43d0-89e8-0b6073fb1e2a"
-					(reference "#PWR017")
-					(unit 1)
-				)
-			)
-		)
-	)
-	(symbol
 		(lib_id "power:VCC")
 		(at 120.65 64.77 0)
@@
 			)
 		)
-		(property "Value" "5.1k"
+		(property "Value" "56k"
 			(at 110.49 71.882 90)
 			(effects
@@
 			)
 		)
-		(property "Value" "5.1k"
+		(property "Value" "56k"
 			(at 110.49 77.978 90)
 			(effects
